File: electrical/nuc980-poc1.kicad_sch (KiCad schematic)
At the start: 110 parts, among them J2 5-6VDC in, J3 JTAG, J4 Serial FTDI Header, J5 USB-A, Q1 MMBT3904, SW1 User Button, SW2 Boot Source, SW3 Reset, U1 PAM2306AYPKE, U2 LM3670MF, U3 W25Q128JVS, U4 NUC980DR61YC, Y1 12 MHz

Commit message: Add SD card to NUC980 dev board (#3)
Signed-off-by: nbpion <87685723+nbpion@users.noreply.github.com>
Parts:
- added J5: Conn_01x08, Connector_PinHeader_2.54mm:PinHeader_1x08_P2.54mm_Vertical, symbol Connector_Generic:Conn_01x08
- added J6: Molex MicroSD 503182-1852, SnapEDA:MOLEX_503182-1852, symbol SnapEDA:Molex 503182-1852
- U2: renamed from U3; Comment Flash ROM -> SPI NOR
- renumbered C15 to C11, C16 to C12, C17 to C13, C18 to C14, C11 to C15, C12 to C16, C13 to C17, C14 to C18, J2 to J1, J3 to J2, J4 to J3, J5 to J4, R8 to R5, R5 to R6, R6 to R7, R7 to R8, TP13 to TP10, TP8 to TP11, TP9 to TP12, TP10 to TP13, TP25 to TP19, TP26 to TP20, TP19 to TP21, TP20 to TP22, TP21 to TP23, TP22 to TP24, TP23 to TP25, TP24 to TP26, TP11 to TP8, TP12 to TP9, U2 to U3
Connections:
- net +3V3: now also J5.5 (Pin_5), J6.4 (VDD)
- net Earth: now also J5.3 (Pin_3), J6.6 (VSS), J6.P1 (SHIELD), J6.P2 (SHIELD), J6.P3 (SHIELD), J6.P4 (SHIELD), J6.P5 (SHIELD)
- net at TP4.1, U2.5 (DI(IO0)): now also RN2.8 (R1.2); no longer RN2.5 (R4.2)
- net at R1.1, TP1.1, U2.1 (~CS): now also RN2.5 (R4.2); no longer RN2.8 (R1.2)
- net at U4.33 (PD.2): now also RN2.4 (R4.1); no longer RN2.1 (R1.1)
- net at U4.34 (PD.3): now also RN2.3 (R3.1); no longer RN2.2 (R2.1)
- net at U4.35 (PD.4): now also RN2.2 (R2.1); no longer RN2.3 (R3.1)
- net at U4.36 (PD.5): now also RN2.1 (R1.1); no longer RN2.4 (R4.1)
- net SD1_CMD: now reaches U4.41 (PF.0)
- net SD1_CMD: now also J5.6 (Pin_6), J6.3 (CMD)
- net SD1_CLK: now reaches U4.42 (PF.1)
- net SD1_CLK: now also J5.4 (Pin_4), J6.5 (CLK)
- net SD1_D0: now reaches U4.43 (PF.2)
- net SD1_D0: now also J5.2 (Pin_2), J6.7 (DAT0)
- net SD1_D1: now reaches U4.44 (PF.3)
- net SD1_D1: now also J5.1 (Pin_1), J6.8 (DAT1)
- net SD1_D2: now reaches U4.45 (PF.4)
- net SD1_D2: now also J5.8 (Pin_8), J6.1 (DATA2)
- net SD1_D3: now reaches U4.46 (PF.5)
- net SD1_D3: now also J5.7 (Pin_7), J6.2 (CD/DAT3)
- net SD1_~{CD}: now reaches U4.47 (PF.6)
- net SD1_~{CD}: now also J6.DT (DETECT)
- net at TP2.1, U2.6 (CLK): now also RN2.6 (R3.2); no longer RN2.7 (R2.2)
- net at TP3.1, U2.2 (DO(IO1)): now also RN2.7 (R2.2); no longer RN2.6 (R3.2)
- no-connect marks 26 -> 20
Other:
- note added: "SparkFun MicroSD breakout: Breakout Pin <-> SD Card Pin 1/RS = 8/D1 2/DO = 7/D0 3/GND = 6/GND 4/CLK = 5/CLK 5/VCC = 4/VDD 6/DI = 3/CMD 7/CS = 2/D3 8/RS = 1/D2"
- moved on the sheet: C10, C11, C12, C13, C14, C5, C6, C9, D1, D2, F1, FB4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
